File: v1/plate/pcb_plate/tif.sch (KiCad schematic (older format))
At the start: 99 parts, among them J2 MJ-4PP-9, J3 OLED, SW10A1 SW_PUSH, SW10B1 SW_PUSH, SW11A1 SW_PUSH, SW11B1 SW_PUSH, SW12A1 SW_PUSH, SW12B1 SW_PUSH, SW13A1 SW_PUSH, SW13B1 SW_PUSH, SW14A1 SW_PUSH, SW14B1 SW_PUSH, SW15A1 SW_PUSH, SW15B1 SW_PUSH, SW16A1 SW_PUSH, SW16B1 SW_PUSH, SW17A1 SW_PUSH, SW17B1 SW_PUSH, SW18A1 SW_PUSH, SW18B1 SW_PUSH, SW19A1 SW_PUSH, SW19B1 SW_PUSH, SW1A1 SW_PUSH, SW1B1 SW_PUSH, SW20A1 SW_PUSH, SW20B1 SW_PUSH, SW21A1 SW_PUSH, SW21B1 SW_PUSH, SW22A1 SW_PUSH, SW22B1 SW_PUSH, SW23 Rotary_Encoder_Switch, SW24A1 SW_PUSH, SW24B1 SW_PUSH, SW25A1 SW_PUSH, SW25B1 SW_PUSH, SW26A1 SW_PUSH, SW26B1 SW_PUSH, SW2A1 SW_PUSH, SW2B1 SW_PUSH, SW3A1 SW_PUSH, SW3B1 SW_PUSH, SW4A1 SW_PUSH, SW4B1 SW_PUSH, SW5A1 SW_PUSH, SW5B1 SW_PUSH, SW6A1 SW_PUSH, SW6B1 SW_PUSH, SW7A1 SW_PUSH, SW7B1 SW_PUSH, SW8A1 SW_PUSH, SW8B1 SW_PUSH, SW9A1 SW_PUSH, SW9B1 SW_PUSH, U1 ProMicro

Commit message: finished top plate switch mounts, switched holes on plate
Parts:
- H1, H2, H3, H4, H5, H6: footprint SofleKeyboard-footprint:HOLE_M2_TH -> SofleKeyboard-footprint:M2_HOLE_PCB
Changed lines of the file:
@@
 F 0 "H1" H 6186 6053 60  0000 L CNN
 F 1 "Hole" H 6186 5947 60  0000 L CNN
-F 2 "SofleKeyboard-footprint:HOLE_M2_TH" H 6000 6000 60  0001 C CNN
+F 2 "SofleKeyboard-footprint:M2_HOLE_PCB" H 6000 6000 60  0001 C CNN
 F 3 "" H 6000 6000 60  0001 C CNN
 	1    6000 6000
@@
 F 0 "H2" H 6786 6053 60  0000 L CNN
 F 1 "Hole" H 6786 5947 60  0000 L CNN
-F 2 "SofleKeyboard-footprint:HOLE_M2_TH" H 6600 6000 60  0001 C CNN
+F 2 "SofleKeyboard-footprint:M2_HOLE_PCB" H 6600 6000 60  0001 C CNN
 F 3 "" H 6600 6000 60  0001 C CNN
 	1    6600 6000
@@
 F 0 "H3" H 7386 6053 60  0000 L CNN
 F 1 "Hole" H 7386 5947 60  0000 L CNN
-F 2 "SofleKeyboard-footprint:HOLE_M2_TH" H 7200 6000 60  0001 C CNN
+F 2 "SofleKeyboard-footprint:M2_HOLE_PCB" H 7200 6000 60  0001 C CNN
 F 3 "" H 7200 6000 60  0001 C CNN
 	1    7200 6000
@@
 F 0 "H4" H 7986 6053 60  0000 L CNN
 F 1 "Hole" H 7986 5947 60  0000 L CNN
-F 2 "SofleKeyboard-footprint:HOLE_M2_TH" H 7800 6000 60  0001 C CNN
+F 2 "SofleKeyboard-footprint:M2_HOLE_PCB" H 7800 6000 60  0001 C CNN
 F 3 "" H 7800 6000 60  0001 C CNN
 	1    7800 6000
@@
 F 0 "H5" H 8586 6053 60  0000 L CNN
 F 1 "Hole" H 8586 5947 60  0000 L CNN
-F 2 "SofleKeyboard-footprint:HOLE_M2_TH" H 8400 6000 60  0001 C CNN
+F 2 "SofleKeyboard-footprint:M2_HOLE_PCB" H 8400 6000 60  0001 C CNN
 F 3 "" H 8400 6000 60  0001 C CNN
 	1    8400 6000
@@
 F 0 "H6" H 9186 6053 60  0000 L CNN
 F 1 "Hole" H 9186 5947 60  0000 L CNN
-F 2 "SofleKeyboard-footprint:HOLE_M2_TH" H 9000 6000 60  0001 C CNN
+F 2 "SofleKeyboard-footprint:M2_HOLE_PCB" H 9000 6000 60  0001 C CNN
 F 3 "" H 9000 6000 60  0001 C CNN
 	1    9000 6000
