File: v1/plate/pcb_plate/tif.kicad_pcb (KiCad board)
At the start: 2 copper layers, 161.7 x 126 mm, 22 parts, among them J2 MJ-4PP-9, U1 ProMicro

Commit message: top plate finished
Parts:
- removed H7, H8: Hole, SofleKeyboard-footprint:M2_HOLE_PCB
- removed J2: MJ-4PP-9, kbd:MJ-4PP-9
- removed JP1, JP8: GND, SofleKeyboard-footprint:Jumper
- removed JP2, JP7: VCC, SofleKeyboard-footprint:Jumper
- removed JP3, JP6: SCL, SofleKeyboard-footprint:Jumper
- removed JP4, JP5: SDA, SofleKeyboard-footprint:Jumper
- removed OLED: OLED, SofleKeyboard-footprint:OLED_4Pin
- removed R1, R2: R, SofleKeyboard-footprint:R_1206_DoubleSided
- removed RSW1: SW_RST, footprints:SW_PUSH_6mm
- removed U1: ProMicro, Keebio-Parts:ArduinoProMicro
Routing:
- net GND: track 87.4 -> 0.00 mm, vias 2 -> 0
- net VCC: track 39.5 -> 0.00 mm, vias 1 -> 0
- net SDA: track 36.7 -> 0.00 mm, vias 2 -> 0
- net COL4: track 36.4 -> 0.00 mm
- net COL3: track 30.7 -> 0.00 mm
- net COL2: track 28.7 -> 0.00 mm
- net DATA: track 28.2 -> 0.00 mm
- net COL1: track 26.6 -> 0.00 mm
- net SCL: track 23.1 -> 0.00 mm, vias 1 -> 0
- net RESET: track 17.1 -> 0.00 mm
- net ENCA: track 4.76 -> 0.00 mm
- net Net-(J3-Pad4): track 4.50 -> 0.00 mm, vias 1 -> 0
- net Net-(J3-Pad3): track 4.50 -> 0.00 mm, vias 1 -> 0
- net Net-(J3-Pad2): track 4.50 -> 0.00 mm, vias 1 -> 0
- net Net-(J3-Pad1): track 4.50 -> 0.00 mm, vias 1 -> 0
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Other:
- outline, holes or cut-outs redrawn
